File: Hardware/KiCad/controle-v1.0.0/controle-v1.0.0.kicad_sch (KiCad schematic)
At the start: 11 parts, among them J1 Gravador, J2 JTAG, SW1 BOOT, SW2 EN, U1 ESP32-S3

Commit message: feat: Hardware
Criando estrutura de projeto, e adicionando esquema ESP32-S3
Parts:
- removed C1, C2, C3: 100nF, Capacitor_SMD:C_0805_2012Metric, symbol Device:C
- removed J1: Gravador, Connector_PinHeader_2.54mm:PinHeader_1x04_P2.54mm_Vertical, symbol Connector:Conn_01x04_Male
- removed J2: JTAG, Connector_PinHeader_2.54mm:PinHeader_2x03_P2.54mm_Vertical, symbol Connector_Generic:Conn_02x03_Counter_Clockwise
- removed R1, R2: 1K5, Resistor_SMD:R_0805_2012Metric, symbol Device:R
- removed R3: 10K, Resistor_SMD:R_0805_2012Metric, symbol Device:R
- removed SW1: BOOT, Button_Switch_THT:SW_PUSH_6mm_H4.3mm, symbol Switch:SW_MEC_5E
- removed SW2: EN, Button_Switch_THT:SW_PUSH_6mm_H4.3mm, symbol Switch:SW_MEC_5E
- removed U1: ESP32-S3, A.R.footprints:ESP32_S3_WROOM_1_N16, symbol A.R.shematic:ESP32_S3_WROOM_1_N16
Other:
- added sheet Fonte (Fonte.kicad_sch)
- added sheet Input (Input.kicad_sch)
- added sheet MCU (MCU.kicad_sch)
- added sheet Módulos (Módulos.kicad_sch)
- note removed: "ESP32 S3 - Wroom"
- note removed: "I2C"
- note removed: "JTAG"
- note removed: "MTCK"
- note removed: "MTDI"
- note removed: "MTDO"
- note removed: "MTMS"
- note removed: "Não usar"
- note removed: "SCL"
- note removed: "SDA"
